Commit message: remove gazebo sim in control xacro

File: description/ros2_control.xacro (robot description, xacro)
@@ -1,5 +1,4 @@
 <?xml version="1.0"?>
 <robot xmlns:xacro="http://www.ros.org/wiki/xacro">
-  <!-- <xacro:unless value="$(arg sim_mode)"> -->
         <ros2_control name="RealRobot" type="system">
             <hardware>
@@ -30,28 +29,4 @@
             </joint>
         </ros2_control>
-  <!--   </xacro:unless> -->
-   <!--  <xacro:if value="$(arg sim_mode)">
-        <ros2_control name="GazeboSystem" type="system">
-            <hardware>
-                <plugin>gazebo_ros2_control/GazeboSystem</plugin>
-            </hardware>
-            <joint name="left_wheel_joint">
-                <command_interface name="velocity">
-                    <param name="min">-10</param>
-                    <param name="max">10</param>
-                </command_interface>
-                <state_interface name="velocity"/>
-                <state_interface name="position"/>
-            </joint>
-            <joint name="right_wheel_joint">
-                <command_interface name="velocity">
-                    <param name="min">-10</param>
-                    <param name="max">10</param>
-                </command_interface>
-                <state_interface name="velocity"/>
-                <state_interface name="position"/>
-            </joint>
-        </ros2_control>
-   </xacro:if> -->
     <gazebo>
         <plugin name="gazebo_ros2_control" filename="libgazebo_ros2_control.so">

Commit message: Fix gazebo

File: description/ros2_control.xacro (robot description, xacro)
@@ -1,4 +1,5 @@
 <?xml version="1.0"?>
 <robot xmlns:xacro="http://www.ros.org/wiki/xacro">
+    <xacro:unless value="$(arg sim_mode)">
         <ros2_control name="RealRobot" type="system">
             <hardware>
@@ -29,8 +30,32 @@
             </joint>
         </ros2_control>
+    </xacro:unless>
+<xacro:if value="$(arg sim_mode)">
+        <ros2_control name="GazeboSystem" type="system">
+            <hardware>
+                <plugin>gazebo_ros2_control/GazeboSystem</plugin>
+            </hardware>
+            <joint name="left_wheel_joint">
+                <command_interface name="velocity">
+                    <param name="min">-10</param>
+                    <param name="max">10</param>
+                </command_interface>
+                <state_interface name="velocity"/>
+                <state_interface name="position"/>
+            </joint>
+            <joint name="right_wheel_joint">
+                <command_interface name="velocity">
+                    <param name="min">-10</param>
+                    <param name="max">10</param>
+                </command_interface>
+                <state_interface name="velocity"/>
+                <state_interface name="position"/>
+            </joint>
+        </ros2_control>
+    </xacro:if>
     <gazebo>
         <plugin name="gazebo_ros2_control" filename="libgazebo_ros2_control.so">
             <parameters>$(find my_bot)/config/my_controllers.yaml</parameters>
-         <!--   <parameters>$(find my_bot)/config/gaz_ros2_ctl_use_sim.yaml</parameters> -->
+         <parameters>$(find my_bot)/config/gaz_ros2_ctl_use_sim.yaml</parameters>
          </plugin>
     </gazebo>

Commit message: gaz ros control add

File: description/ros2_control.xacro (robot description, xacro)
@@ -31,30 +31,30 @@
         </ros2_control>
     </xacro:unless>
-<xacro:if value="$(arg sim_mode)">
+    <xacro:if value="$(arg sim_mode)">
         <ros2_control name="GazeboSystem" type="system">
-            <hardware>
-                <plugin>gazebo_ros2_control/GazeboSystem</plugin>
-            </hardware>
-            <joint name="left_wheel_joint">
-                <command_interface name="velocity">
-                    <param name="min">-10</param>
-                    <param name="max">10</param>
-                </command_interface>
-                <state_interface name="velocity"/>
-                <state_interface name="position"/>
-            </joint>
-            <joint name="right_wheel_joint">
-                <command_interface name="velocity">
-                    <param name="min">-10</param>
-                    <param name="max">10</param>
-                </command_interface>
-                <state_interface name="velocity"/>
-                <state_interface name="position"/>
-            </joint>
+                <hardware>
+                    <plugin>gazebo_ros2_control/GazeboSystem</plugin>
+                </hardware>
+                <joint name="left_wheel_joint">
+                    <command_interface name="velocity">
+                        <param name="min">-10</param>
+                        <param name="max">10</param>
+                    </command_interface>
+                    <state_interface name="velocity"/>
+                    <state_interface name="position"/>
+                </joint>
+                <joint name="right_wheel_joint">
+                    <command_interface name="velocity">
+                        <param name="min">-10</param>
+                        <param name="max">10</param>
+                    </command_interface>
+                    <state_interface name="velocity"/>
+                    <state_interface name="position"/>
+                </joint>
         </ros2_control>
     </xacro:if>
     <gazebo>
         <plugin name="gazebo_ros2_control" filename="libgazebo_ros2_control.so">
-            <parameters>$(find my_bot)/config/my_controllers.yaml</parameters>
+         <parameters>$(find my_bot)/config/my_controllers.yaml</parameters>
          <parameters>$(find my_bot)/config/gaz_ros2_ctl_use_sim.yaml</parameters>
          </plugin>
